Commit message: Update baxter URDF

File: urdf/baxter.urdf (robot description, URDF)
Before this commit: robot baxter, 49 links, 48 joints
Links:
- added link l_gripper_l_finger, mass 0.02; collision box size=0.01 0.0135 0.1127; collision box size=0.01 0.05 0.017
- added link l_gripper_l_finger_tip, mass 0.01; collision box size=0.042 0.0065 0.037; visual mesh filename=package://rethink_ee_description/meshes/electric_gripper/fi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
- added link l_gripper_r_finger, mass 0.02; collision box size=0.01 0.0135 0.1127; collision box size=0.01 0.05 0.017
- added link l_gripper_r_finger_tip, mass 0.01; collision box size=0.042 0.0065 0.037; visual mesh filename=package://rethink_ee_description/meshes/electric_gripper/fi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
- added link r_gripper_l_finger, mass 0.02; collision box size=0.01 0.0135 0.1127; collision box size=0.01 0.05 0.017
- added link r_gripper_l_finger_tip, mass 0.01; collision cylinder length=0.037 radius=0.008; visual mesh filename=package://rethink_ee_description/meshes/electric_gripper/fi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
- added link r_gripper_r_finger, mass 0.02; collision box size=0.01 0.0135 0.1127; collision box size=0.01 0.05 0.017
- added link r_gripper_r_finger_tip, mass 0.01; collision cylinder length=0.037 radius=0.008; visual mesh filename=package://rethink_ee_description/meshes/electric_gripper/fi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
- link left_gripper: geometry 
- link left_gripper_base: mass 0.0001 -> 0.3; geometry collision cylinder length=0.1 radius=0.029; visual mesh filename=package://rethink_ee_description/meshes/electric_gripper/el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
- link right_gripper: geometry 
- link right_gripper_base: mass 0.0001 -> 0.3; geometry collision cylinder length=0.1 radius=0.029; visual mesh filename=package://rethink_ee_description/meshes/electric_gripper/el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
Joints:
- added joint l_gripper_l_finger_joint: type prismatic, parent left_gripper_base, child l_gripper_l_finger, origin xyz=0.0 -0.0015 0.02 rpy=0 0 0, axis 0 1 0, limit lower=0.0 upper=0.020833 effort=20.0 velocity=5.0
- added joint l_gripper_l_finger_tip_joint: type fixed, parent l_gripper_l_finger, child l_gripper_l_finger_tip, origin xyz=0.0 0.01725 0.1127 rpy=0 0 0
- added joint l_gripper_r_finger_joint: type prismatic, parent left_gripper_base, child l_gripper_r_finger, origin xyz=0.0 0.0015 0.02 rpy=0 0 0, axis 0 1 0, limit lower=-0.020833 upper=0.0 effort=20.0 velocity=5.0, mimic joint=l_gripper_l_finger_joint multiplier=-1.0
- added joint l_gripper_r_finger_tip_joint: type fixed, parent l_gripper_r_finger, child l_gripper_r_finger_tip, origin xyz=0.0 -0.01725 0.1127 rpy=0 0 0
- added joint r_gripper_l_finger_joint: type prismatic, parent right_gripper_base, child r_gripper_l_finger, origin xyz=0.0 -0.0015 0.02 rpy=0 0 0, axis 0 1 0, limit lower=0.0 upper=0.020833 effort=20.0 velocity=5.0
- added joint r_gripper_l_finger_tip_joint: type fixed, parent r_gripper_l_finger, child r_gripper_l_finger_tip, origin xyz=0.0 0.01725 0.1127 rpy=0 0 0
- added joint r_gripper_r_finger_joint: type prismatic, parent right_gripper_base, child r_gripper_r_finger, origin xyz=0.0 0.0015 0.02 rpy=0 0 0, axis 0 1 0, limit lower=-0.020833 upper=0.0 effort=20.0 velocity=5.0, mimic joint=r_gripper_l_finger_joint multiplier=-1.0
- added joint r_gripper_r_finger_tip_joint: type fixed, parent r_gripper_r_finger, child r_gripper_r_finger_tip, origin xyz=0.0 -0.01725 0.1127 rpy=0 0 0
- joint head_pan: limit lower=-1.57079632679 upper=1.57079632679 effort=50000 velocity=10000 -> lower=-1.3963 upper=1.3963 effort=50000 velocity=10000
- joint left_endpoint: origin xyz=0.0 0 0.025 rpy=0 0 0 -> xyz=0 0 0.1327 rpy=0 0 0
- joint left_gripper_base: origin xyz=0 0 0 rpy=0 0 0 -> xyz=0 0 0.025 rpy=0 0 0
- joint left_s1: limit lower=-2.147 upper=1.047 effort=100.0 velocity=1.5 -> lower=-2.147 upper=1.047 effort=50.0 velocity=1.5
- joint right_endpoint: origin xyz=0.0 0 0.025 rpy=0 0 0 -> xyz=0 0 0.1327 rpy=0 0 0
- joint right_gripper_base: origin xyz=0 0 0 rpy=0 0 0 -> xyz=0 0 0.025 rpy=0 0 0
- joint right_s1: limit lower=-2.147 upper=1.047 effort=100.0 velocity=1.5 -> lower=-2.147 upper=1.047 effort=50.0 velocity=1.5

Commit message: [urdf] Rename some links and joints so that they have different names
  - head_camera -> head_camera_[link|joint],
  - left_hand -> left_hand_[link|joint],
  - right_hand -> right_hand_[link|joint],
  - left_hand_camera -> left_hand_camera_[link|joint],
  - right_hand_camera -> right_hand_camera_[link|joint],
  - left_hand_camera_axis -> left_hand_camera_axis_[link|joint],
  - right_hand_camera_axis -> right_hand_camera_axis_[link|joint],
  - left_gripper_base -> left_gripper_base_[link|joint],
  - right_gripper_base -> right_gripper_base_[link|joint],
  - left_hand_accelerometer -> left_hand_accelerometer_[link|joint],
  - right_hand_accelerometer -> right_hand_accelerometer_[link|joint],
  - left_hand_range -> left_hand_range_[link|joint],
  - right_hand_range -> right_hand_range_[link|joint],

File: urdf/baxter.urdf (robot description, URDF)
Before this commit: robot baxter, 57 links, 56 joints
Links:
- removed link head_camera
- removed link left_gripper_base
- removed link left_hand
- removed link left_hand_accelerometer
- removed link left_hand_camera
- removed link left_hand_camera_axis
- removed link left_hand_range
- removed link right_gripper_base
- removed link right_hand
- removed link right_hand_accelerometer
- removed link right_hand_camera
- removed link right_hand_camera_axis
- removed link right_hand_range
- added link head_camera_link, mass 0.0001
- added link left_gripper_base_link, mass 0.3; collision cylinder length=0.1 radius=0.029; visual mesh filename=package://rethink_ee_description/meshes/electric_gripper/el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
- added link left_hand_accelerometer_link, mass 0.0001; visual box size=0.01 0.01 0.01
- added link left_hand_camera_axis_link, mass 0.0001
- added link left_hand_camera_link, mass 0.0001; visual cylinder length=0.01 radius=0.02
- added link left_hand_link, mass 0.19125; collision cylinder length=0.0464 radius=0.04
- added link left_hand_range_link, mass 0.0001; visual box size=0.005 .02 .005
- added link right_gripper_base_link, mass 0.3; collision cylinder length=0.1 radius=0.029; visual mesh filename=package://rethink_ee_description/meshes/electric_gripper/el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
- added link right_hand_accelerometer_link, mass 0.0001; visual box size=0.01 0.01 0.01
- added link right_hand_camera_axis_link, mass 0.0001
- added link right_hand_camera_link, mass 0.0001; visual cylinder length=0.01 radius=0.02
- added link right_hand_link, mass 0.19125; collision cylinder length=0.0464 radius=0.04
- added link right_hand_range_link, mass 0.0001; visual box size=0.005 .02 .005
Joints:
- removed joint head_camera
- removed joint left_gripper_base
- removed joint left_hand
- removed joint left_hand_accelerometer
- removed joint left_hand_camera
- removed joint left_hand_camera_axis
- removed joint left_hand_range
- removed joint right_gripper_base
- removed joint right_hand
- removed joint right_hand_accelerometer
- removed joint right_hand_camera
- removed joint right_hand_camera_axis
- removed joint right_hand_range
- added joint head_camera_joint: type fixed, parent head, child head_camera_link, origin xyz=0.12839 0 0.06368 rpy=1.75057 0 1.57079632679
- added joint left_gripper_base_joint: type fixed, parent left_hand_link, child left_gripper_base_link, origin xyz=0 0 0.025 rpy=0 0 0
- added joint left_hand_accelerometer_joint: type fixed, parent left_hand_link, child left_hand_accelerometer_link, origin xyz=0.00198 0.000133 -0.0146 rpy=0 0 0
- added joint left_hand_camera_axis_joint: type fixed, parent left_hand_link, child left_hand_camera_axis_link, origin xyz=0.03825 0.012 0.015355 rpy=0 0 0
- added joint left_hand_camera_joint: type fixed, parent left_hand_link, child left_hand_camera_link, origin xyz=0.03825 0.012 0.015355 rpy=0 0 -1.57079633
- added joint left_hand_joint: type fixed, parent left_wrist, child left_hand_link, origin xyz=0 0 0.11355 rpy=0 0 0, axis 0 0 1
- added joint left_hand_range_joint: type fixed, parent left_hand_link, child left_hand_range_link, origin xyz=0.032 -0.020245 0.0288 rpy=0 -1.57079632679 -1.57079632679
- added joint right_gripper_base_joint: type fixed, parent right_hand_link, child right_gripper_base_link, origin xyz=0 0 0.025 rpy=0 0 0
- added joint right_hand_accelerometer_joint: type fixed, parent right_hand_link, child right_hand_accelerometer_link, origin xyz=0.00198 0.000133 -0.0146 rpy=0 0 0
- added joint right_hand_camera_axis_joint: type fixed, parent right_hand_link, child right_hand_camera_axis_link, origin xyz=0.03825 0.012 0.015355 rpy=0 0 0
- added joint right_hand_camera_joint: type fixed, parent right_hand_link, child right_hand_camera_link, origin xyz=0.03825 0.012 0.015355 rpy=0 0 -1.57079633
- added joint right_hand_joint: type fixed, parent right_wrist, child right_hand_link, origin xyz=0 0 0.11355 rpy=0 0 0, axis 0 0 1
- added joint right_hand_range_joint: type fixed, parent right_hand_link, child right_hand_range_link, origin xyz=0.032 -0.020245 0.0288 rpy=0 -1.57079632679 -1.57079632679
- joint l_gripper_l_finger_joint: parent left_gripper_base -> left_gripper_base_link
- joint l_gripper_r_finger_joint: parent left_gripper_base -> left_gripper_base_link
- joint left_endpoint: parent left_gripper_base -> left_gripper_base_link
- joint r_gripper_l_finger_joint: parent right_gripper_base -> right_gripper_base_link
- joint r_gripper_r_finger_joint: parent right_gripper_base -> right_gripper_base_link
- joint right_endpoint: parent right_gripper_base -> right_gripper_base_link

File: urdf/baxter_colman.urdf (robot description, URDF)
Before this commit: robot baxter, 54 links, 53 joints
Links:
- removed link head_camera
- removed link left_gripper_base
- removed link left_hand
- removed link left_hand_accelerometer
- removed link left_hand_camera
- removed link left_hand_camera_axis
- removed link left_hand_range
- removed link right_gripper_base
- removed link right_hand
- removed link right_hand_camera
- removed link right_hand_camera_axis
- removed link right_hand_range
- added link head_camera_link, mass 0.0001
- added link left_gripper_base_link, mass 0.0001; visual box size=0.025 0.075 0.035
- added link left_hand_accelerometer_link, mass 0.0001; visual box size=0.01 0.01 0.01
- added link left_hand_camera_axis_link, mass 0.0001
- added link left_hand_camera_link, mass 0.0001; visual cylinder length=0.01 radius=0.02
- added link left_hand_link, mass 0.19125; collision cylinder length=0.0464 radius=0.04
- added link left_hand_range_link, mass 0.0001; visual box size=0.005 .02 .005
- added link right_gripper_base_link, mass 0.0001; visual box size=0.025 0.075 0.035
- added link right_hand_camera_axis_link, mass 0.0001
- added link right_hand_camera_link, mass 0.0001; visual cylinder length=0.01 radius=0.02
- added link right_hand_link, mass 0.19125; collision cylinder length=0.0464 radius=0.04
- added link right_hand_range_link, mass 0.0001; visual box size=0.005 .02 .005
Joints:
- removed joint head_camera
- removed joint left_gripper_base
- removed joint left_hand
- removed joint left_hand_accelerometer
- removed joint left_hand_camera
- removed joint left_hand_camera_axis
- removed joint left_hand_range
- removed joint right_gripper_base
- removed joint right_hand
- removed joint right_hand_camera
- removed joint right_hand_camera_axis
- removed joint right_hand_range
- added joint head_camera_joint: type fixed, parent head, child head_camera_link, origin xyz=0.12839 0 0.06368 rpy=1.75057 0 1.57079632679
- added joint left_gripper_base_joint: type fixed, parent left_hand_link, child left_gripper_base_link, origin xyz=0 0 0 rpy=0 0 0
- added joint left_hand_accelerometer_joint: type fixed, parent left_hand_link, child left_hand_accelerometer_link, origin xyz=0.00198 0.000133 -0.0146 rpy=0 0 0
- added joint left_hand_camera_axis_joint: type fixed, parent left_hand_link, child left_hand_camera_axis_link, origin xyz=0.03825 0.012 0.015355 rpy=0 0 0
- added joint left_hand_camera_joint: type fixed, parent left_hand_link, child left_hand_camera_link, origin xyz=0.03825 0.012 0.015355 rpy=0 0 -1.57079633
- added joint left_hand_joint: type fixed, parent left_wrist, child left_hand_link, origin xyz=0 0 0.11355 rpy=0 0 0, axis 0 0 1
- added joint left_hand_range_joint: type fixed, parent left_hand_link, child left_hand_range_link, origin xyz=0.032 -0.020245 0.0288 rpy=0 -1.57079632679 -1.57079632679
- added joint right_gripper_base_joint: type fixed, parent right_hand_link, child right_gripper_base_link, origin xyz=0 0 0 rpy=0 0 0
- added joint right_hand_camera_axis_joint: type fixed, parent right_hand_link, child right_hand_camera_axis_link, origin xyz=0.03825 0.012 0.015355 rpy=0 0 0
- added joint right_hand_camera_joint: type fixed, parent right_hand_link, child right_hand_camera_link, origin xyz=0.03825 0.012 0.015355 rpy=0 0 -1.57079633
- added joint right_hand_joint: type fixed, parent right_wrist, child right_hand_link, origin xyz=0 0 0.11355 rpy=0 0 0, axis 0 0 1
- added joint right_hand_range_joint: type fixed, parent right_hand_link, child right_hand_range_link, origin xyz=0.032 -0.020245 0.0288 rpy=0 -1.57079632679 -1.57079632679
- joint left_endpoint: parent left_gripper_base -> left_gripper_base_link
- joint right_endpoint: parent right_gripper_base -> right_gripper_base_link

Commit message: Add Baxter meshes since robot is deprecated
  - useful for benchmark

File: urdf/baxter.urdf (robot description, URDF)
Before this commit: robot baxter, 57 links, 56 joints
Links:
- link head: geometry collision sphere radius=0.001; visual mesh filename=package://hpp-baxter/meshes/head/H0.DAE
- link l_gripper_l_finger: geometry collision box size=0.01 0.0135 0.1127; collision box size=0.01 0.05 0.017
- link l_gripper_l_finger_tip: geometry collision box size=0.042 0.0065 0.037; visual mesh filename=package://hpp-baxter/meshes/electric_gripper/fingers/paddle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
- link l_gripper_r_finger: geometry collision box size=0.01 0.0135 0.1127; collision box size=0.01 0.05 0.017
- link l_gripper_r_finger_tip: geometry collision box size=0.042 0.0065 0.037; visual mesh filename=package://hpp-baxter/meshes/electric_gripper/fingers/paddle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
- link left_gripper_base_link: geometry collision cylinder length=0.1 radius=0.029; visual mesh filename=package://hpp-baxter/meshes/electric_gripper/electric_gripp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
- link left_lower_elbow: geometry collision cylinder length=0.10 radius=0.06; visual mesh filename=package://hpp-baxter/meshes/lower_elbow/E1.DAE
- link left_lower_forearm: geometry collision cylinder length=0.10 radius=0.06; visual mesh filename=package://hpp-baxter/meshes/lower_forearm/W1.DAE
- link left_lower_shoulder: geometry collision cylinder length=0.12 radius=0.06; visual mesh filename=package://hpp-baxter/meshes/lower_shoulder/S1.DAE
- link left_upper_elbow: geometry collision cylinder length=0.107 radius=0.06; visual mesh filename=package://hpp-baxter/meshes/upper_elbow/E0.DAE
- link left_upper_forearm: geometry collision cylinder length=0.088 radius=0.06; visual mesh filename=package://hpp-baxter/meshes/upper_forearm/W0.DAE
- link left_upper_shoulder: geometry collision cylinder length=0.2722 radius=0.06; visual mesh filename=package://hpp-baxter/meshes/upper_shoulder/S0.DAE
- link left_wrist: geometry collision cylinder length=0.165 radius=0.06; visual mesh filename=package://hpp-baxter/meshes/wrist/W2.DAE
- link pedestal: geometry collision mesh filename=package://hpp-baxter/meshes/base/pedestal_link_collision.DAE; visual mesh filename=package://hpp-baxter/meshes/base/PEDESTAL.DAE
- link r_gripper_l_finger: geometry collision box size=0.01 0.0135 0.1127; collision box size=0.01 0.05 0.017
- link r_gripper_l_finger_tip: geometry collision cylinder length=0.037 radius=0.008; visual mesh filename=package://hpp-baxter/meshes/electric_gripper/fingers/half_r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
- link r_gripper_r_finger: geometry collision box size=0.01 0.0135 0.1127; collision box size=0.01 0.05 0.017
- link r_gripper_r_finger_tip: geometry collision cylinder length=0.037 radius=0.008; visual mesh filename=package://hpp-baxter/meshes/electric_gripper/fingers/half_r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
- link right_gripper_base_link: geometry collision cylinder length=0.1 radius=0.029; visual mesh filename=package://hpp-baxter/meshes/electric_gripper/electric_gripp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
- link right_lower_elbow: geometry collision cylinder length=0.10 radius=0.06; visual mesh filename=package://hpp-baxter/meshes/lower_elbow/E1.DAE
- link right_lower_forearm: geometry collision cylinder length=0.10 radius=0.06; visual mesh filename=package://hpp-baxter/meshes/lower_forearm/W1.DAE
- link right_lower_shoulder: geometry collision cylinder length=0.12 radius=0.06; visual mesh filename=package://hpp-baxter/meshes/lower_shoulder/S1.DAE
- link right_upper_elbow: geometry collision cylinder length=0.107 radius=0.06; visual mesh filename=package://hpp-baxter/meshes/upper_elbow/E0.DAE
- link right_upper_forearm: geometry collision cylinder length=0.088 radius=0.06; visual mesh filename=package://hpp-baxter/meshes/upper_forearm/W0.DAE
- link right_upper_shoulder: geometry collision cylinder length=0.2722 radius=0.06; visual mesh filename=package://hpp-baxter/meshes/upper_shoulder/S0.DAE
- link right_wrist: geometry collision cylinder length=0.165 radius=0.06; visual mesh filename=package://hpp-baxter/meshes/wrist/W2.DAE
- link screen: geometry collision sphere radius=0.001; visual mesh filename=package://hpp-baxter/meshes/head/H1.DAE
- link torso: geometry collision mesh filename=package://hpp-baxter/meshes/torso/base_link_collision.DAE; visual mesh filename=package://hpp-baxter/meshes/torso/base_link.DAE

File: urdf/baxter_colman.urdf (robot description, URDF)
Before this commit: robot baxter, 54 links, 53 joints
Links:
- link head: geometry collision sphere radius=0.001; visual mesh filename=package://hpp-baxter/meshes/head/H0.DAE
- link left_lower_elbow: geometry collision cylinder length=0.10 radius=0.06; visual mesh filename=package://hpp-baxter/meshes/lower_elbow/E1.DAE
- link left_lower_forearm: geometry collision cylinder length=0.10 radius=0.06; visual mesh filename=package://hpp-baxter/meshes/lower_forearm/W1.DAE
- link left_lower_shoulder: geometry collision cylinder length=0.12 radius=0.06; visual mesh filename=package://hpp-baxter/meshes/lower_shoulder/S1.DAE
- link left_upper_elbow: geometry collision cylinder length=0.107 radius=0.06; visual mesh filename=package://hpp-baxter/meshes/upper_elbow/E0.DAE
- link left_upper_forearm: geometry collision cylinder length=0.088 radius=0.06; visual mesh filename=package://hpp-baxter/meshes/upper_forearm/W0.DAE
- link left_upper_shoulder: geometry collision cylinder length=0.2722 radius=0.06; visual mesh filename=package://hpp-baxter/meshes/upper_shoulder/S0.DAE
- link left_wrist: geometry collision cylinder length=0.165 radius=0.06; visual mesh filename=package://hpp-baxter/meshes/wrist/W2.DAE
- link pedestal: geometry collision box size=0.92 0.83 0.3; visual mesh filename=package://hpp-baxter/meshes/base/PEDESTAL.DAE
- link right_gripper: geometry collision cylinder length=0.1 radius=0.0275; visual mesh filename=package://hpp-baxter/meshes/electric_gripper/electric_gripp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
- link right_gripper_l_finger: geometry collision mesh filename=package://hpp-baxter/meshes/electric_gripper/fingers/standa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; visual mesh filename=package://hpp-baxter/meshes/electric_gripper/fingers/standa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
- link right_gripper_r_finger: geometry collision mesh filename=package://hpp-baxter/meshes/electric_gripper/fingers/standa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; visual mesh filename=package://hpp-baxter/meshes/electric_gripper/fingers/standa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
- link right_lower_elbow: geometry collision cylinder length=0.10 radius=0.06; visual mesh filename=package://hpp-baxter/meshes/lower_elbow/E1.DAE
- link right_lower_forearm: geometry collision cylinder length=0.10 radius=0.06; visual mesh filename=package://hpp-baxter/meshes/lower_forearm/W1.DAE
- link right_lower_shoulder: geometry collision cylinder length=0.12 radius=0.06; visual mesh filename=package://hpp-baxter/meshes/lower_shoulder/S1.DAE
- link right_upper_elbow: geometry collision cylinder length=0.107 radius=0.06; visual mesh filename=package://hpp-baxter/meshes/upper_elbow/E0.DAE
- link right_upper_forearm: geometry collision cylinder length=0.088 radius=0.06; visual mesh filename=package://hpp-baxter/meshes/upper_forearm/W0.DAE
- link right_upper_shoulder: geometry collision cylinder length=0.2722 radius=0.06; visual mesh filename=package://hpp-baxter/meshes/upper_shoulder/S0.DAE
- link right_wrist: geometry collision cylinder length=0.165 radius=0.06; visual mesh filename=package://hpp-baxter/meshes/wrist/W2.DAE
- link screen: geometry collision sphere radius=0.001; visual mesh filename=package://hpp-baxter/meshes/head/H1.DAE
- link torso: geometry collision cylinder length=0.7 radius=0.27; visual mesh filename=package://hpp-baxter/meshes/torso/base_link.DAE
