Commit message: use meshes from example-robot-data

File: urdf/baxter.urdf (robot description, URDF)
Before this commit: robot baxter, 57 links, 56 joints
Links:
- link head: geometry collision sphere radius=0.001; visual mesh filename=package://example-robot-data/robots/baxter_description/mesh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
- link l_gripper_l_finger: geometry collision box size=0.01 0.0135 0.1127; collision box size=0.01 0.05 0.017
- link l_gripper_l_finger_tip: geometry collision box size=0.042 0.0065 0.037; visual mesh filename=package://example-robot-data/robots/baxter_description/mesh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
- link l_gripper_r_finger: geometry collision box size=0.01 0.0135 0.1127; collision box size=0.01 0.05 0.017
- link l_gripper_r_finger_tip: geometry collision box size=0.042 0.0065 0.037; visual mesh filename=package://example-robot-data/robots/baxter_description/mesh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
- link left_gripper_base_link: geometry collision cylinder length=0.1 radius=0.029; visual mesh filename=package://example-robot-data/robots/baxter_description/mesh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
- link left_lower_elbow: geometry collision cylinder length=0.10 radius=0.06; visual mesh filename=package://example-robot-data/robots/baxter_description/mesh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
- link left_lower_forearm: geometry collision cylinder length=0.10 radius=0.06; visual mesh filename=package://example-robot-data/robots/baxter_description/mesh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
- link left_lower_shoulder: geometry collision cylinder length=0.12 radius=0.06; visual mesh filename=package://example-robot-data/robots/baxter_description/mesh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
- link left_upper_elbow: geometry collision cylinder length=0.107 radius=0.06; visual mesh filename=package://example-robot-data/robots/baxter_description/mesh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
- link left_upper_forearm: geometry collision cylinder length=0.088 radius=0.06; visual mesh filename=package://example-robot-data/robots/baxter_description/mesh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
- link left_upper_shoulder: geometry collision cylinder length=0.2722 radius=0.06; visual mesh filename=package://example-robot-data/robots/baxter_description/mesh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
- link left_wrist: geometry collision cylinder length=0.165 radius=0.06; visual mesh filename=package://example-robot-data/robots/baxter_description/mesh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
- link pedestal: geometry collision mesh filename=package://example-robot-data/robots/baxter_description/mesh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; visual mesh filename=package://example-robot-data/robots/baxter_description/mesh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
- link r_gripper_l_finger: geometry collision box size=0.01 0.0135 0.1127; collision box size=0.01 0.05 0.017
- link r_gripper_l_finger_tip: geometry collision cylinder length=0.037 radius=0.008; visual mesh filename=package://example-robot-data/robots/baxter_description/mesh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
- link r_gripper_r_finger: geometry collision box size=0.01 0.0135 0.1127; collision box size=0.01 0.05 0.017
- link r_gripper_r_finger_tip: geometry collision cylinder length=0.037 radius=0.008; visual mesh filename=package://example-robot-data/robots/baxter_description/mesh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
- link right_gripper_base_link: geometry collision cylinder length=0.1 radius=0.029; visual mesh filename=package://example-robot-data/robots/baxter_description/mesh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
- link right_lower_elbow: geometry collision cylinder length=0.10 radius=0.06; visual mesh filename=package://example-robot-data/robots/baxter_description/mesh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
- link right_lower_forearm: geometry collision cylinder length=0.10 radius=0.06; visual mesh filename=package://example-robot-data/robots/baxter_description/mesh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
- link right_lower_shoulder: geometry collision cylinder length=0.12 radius=0.06; visual mesh filename=package://example-robot-data/robots/baxter_description/mesh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
- link right_upper_elbow: geometry collision cylinder length=0.107 radius=0.06; visual mesh filename=package://example-robot-data/robots/baxter_description/mesh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
- link right_upper_forearm: geometry collision cylinder length=0.088 radius=0.06; visual mesh filename=package://example-robot-data/robots/baxter_description/mesh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
- link right_upper_shoulder: geometry collision cylinder length=0.2722 radius=0.06; visual mesh filename=package://example-robot-data/robots/baxter_description/mesh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
- link right_wrist: geometry collision cylinder length=0.165 radius=0.06; visual mesh filename=package://example-robot-data/robots/baxter_description/mesh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
- link screen: geometry collision sphere radius=0.001; visual mesh filename=package://example-robot-data/robots/baxter_description/mesh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
- link torso: geometry collision mesh filename=package://example-robot-data/robots/baxter_description/mesh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; visual mesh filename=package://example-robot-data/robots/baxter_description/mesh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

File: urdf/baxter_colman.urdf (robot description, URDF)
Before this commit: robot baxter, 54 links, 53 joints
Links:
- link head: geometry collision sphere radius=0.001; visual mesh filename=package://example-robot-data/robots/baxter_description/mesh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
- link left_lower_elbow: geometry collision cylinder length=0.10 radius=0.06; visual mesh filename=package://example-robot-data/robots/baxter_description/mesh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
- link left_lower_forearm: geometry collision cylinder length=0.10 radius=0.06; visual mesh filename=package://example-robot-data/robots/baxter_description/mesh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
- link left_lower_shoulder: geometry collision cylinder length=0.12 radius=0.06; visual mesh filename=package://example-robot-data/robots/baxter_description/mesh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
- link left_upper_elbow: geometry collision cylinder length=0.107 radius=0.06; visual mesh filename=package://example-robot-data/robots/baxter_description/mesh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
- link left_upper_forearm: geometry collision cylinder length=0.088 radius=0.06; visual mesh filename=package://example-robot-data/robots/baxter_description/mesh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
- link left_upper_shoulder: geometry collision cylinder length=0.2722 radius=0.06; visual mesh filename=package://example-robot-data/robots/baxter_description/mesh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
- link left_wrist: geometry collision cylinder length=0.165 radius=0.06; visual mesh filename=package://example-robot-data/robots/baxter_description/mesh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
- link pedestal: geometry collision box size=0.92 0.83 0.3; visual mesh filename=package://example-robot-data/robots/baxter_description/mesh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
- link right_gripper: geometry collision cylinder length=0.1 radius=0.0275; visual mesh filename=package://example-robot-data/robots/baxter_description/mesh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
- link right_gripper_l_finger: geometry collision mesh filename=package://example-robot-data/robots/baxter_description/mesh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; visual mesh filename=package://example-robot-data/robots/baxter_description/mesh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
- link right_gripper_r_finger: geometry collision mesh filename=package://example-robot-data/robots/baxter_description/mesh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; visual mesh filename=package://example-robot-data/robots/baxter_description/mesh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
- link right_lower_elbow: geometry collision cylinder length=0.10 radius=0.06; visual mesh filename=package://example-robot-data/robots/baxter_description/mesh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
- link right_lower_forearm: geometry collision cylinder length=0.10 radius=0.06; visual mesh filename=package://example-robot-data/robots/baxter_description/mesh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
- link right_lower_shoulder: geometry collision cylinder length=0.12 radius=0.06; visual mesh filename=package://example-robot-data/robots/baxter_description/mesh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
- link right_upper_elbow: geometry collision cylinder length=0.107 radius=0.06; visual mesh filename=package://example-robot-data/robots/baxter_description/mesh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
- link right_upper_forearm: geometry collision cylinder length=0.088 radius=0.06; visual mesh filename=package://example-robot-data/robots/baxter_description/mesh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
- link right_upper_shoulder: geometry collision cylinder length=0.2722 radius=0.06; visual mesh filename=package://example-robot-data/robots/baxter_description/mesh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
- link right_wrist: geometry collision cylinder length=0.165 radius=0.06; visual mesh filename=package://example-robot-data/robots/baxter_description/mesh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
- link screen: geometry collision sphere radius=0.001; visual mesh filename=package://example-robot-data/robots/baxter_description/mesh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
- link torso: geometry collision cylinder length=0.7 radius=0.27; visual mesh filename=package://example-robot-data/robots/baxter_description/mesh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
